File: pcb2/fakerio2.kicad_pcb (KiCad board)
At the start: 2 copper layers, 99.1 x 49.5 mm, 42 parts, among them J1 Conn_01x03, J2 Conn_01x03, J3 Conn_01x03, J4 Conn_01x03, J5 Conn_01x02, SW1 SW_SPDT_MSM, SW2 SW_SPDT_MSM, SW3 SW_SPDT_MSM, SW4 SW_SPDT_MSM, U1 LM7805_TO220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

Commit message: one more submit before rearranging layout part placement
Parts:
- moved TP6 14.0 mm to (162.6, 109.2)
- moved U1 1.27 mm to (83.8, 108.3)
Other:
- board size 99.1 x 49.5 mm -> 128.3 x 36.8 mm
Changed lines of the file:
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@@
   )
   (footprint "Connector_PinHeader_2.54mm:PinHeader_1x01_P2.54mm_Vertical" (layer "F.Cu")
-    (at 176.53 109.22)
+    (at 162.56 109.22)
     (descr "Through hole straight pin header, 1x01, 2.54mm pitch, single row")
     (tags "Through hole pin header THT 1x01 2.54mm single row")
@@
   )
   (footprint "Package_TO_SOT_THT:TO-220-3_Horizontal_TabDown" (layer "F.Cu")
-    (at 83.82 109.56)
+    (at 83.82 108.29)
     (descr "TO-220-3, Horizontal, RM 2.54mm, see https://www.vishay.com/docs/66542/to-220-1.pdf")
     (tags "TO-220-3 Horizontal RM 2.54mm")
@@
     )
   )
-  (gr_line (start 50.8 63.5) (end 50.8 113.03)
+  (gr_line (start 56.515 111.76) (end 179.07 111.76)
     (stroke (width 0.1) (type default)) (layer "Edge.Cuts"))
-  (gr_line (start 12.7 76.2) (end 111.76 76.2)
+  (gr_line (start 50.8 76.2) (end 50.8 113.03)
+    (stroke (width 0.1) (type default)) (layer "Edge.Cuts"))
+  (gr_line (start 50.8 76.2) (end 179.07 76.2)
+    (stroke (width 0.1) (type default)) (layer "Edge.Cuts"))
+  (gr_line (start 179.07 76.2) (end 179.07 113.03)
     (stroke (width 0.1) (type default)) (layer "Edge.Cuts"))
 )
